Commit message: add bullet demo

File: data/robots/ur10_robotis_d435.urdf (robot description, URDF)
Before this commit: robot ur10_robotis_d435, 19 links, 18 joints
Links:
- link base_link: geometry collision mesh filename=package://ur10/ur10/collision/base.stl; visual mesh filename=package://ur10/ur10/visual/base.dae
- link d435_link: geometry collision box size=0.02505 0.09 0.025; visual mesh filename=package://ur10/realsense2/visual/d435.dae
- link forearm_link: geometry collision mesh filename=package://ur10/ur10/collision/forearm.stl; visual mesh filename=package://ur10/ur10/visual/forearm.dae
- link rh_p12_rn_base: geometry collision mesh filename=package://ur10/robotis_rh_p12_rn/collision/base.stl scale=0.001 0.001 0.001; visual mesh filename=package://ur10/robotis_rh_p12_rn/visual/base.stl scale=0.001 0.001 0.001
- link rh_p12_rn_l1: geometry collision mesh filename=package://ur10/robotis_rh_p12_rn/collision/l1.stl scale=0.001 0.001 0.001; visual mesh filename=package://ur10/robotis_rh_p12_rn/visual/l1.stl scale=0.001 0.001 0.001
- link rh_p12_rn_l2: geometry collision mesh filename=package://ur10/robotis_rh_p12_rn/collision/l2.stl scale=0.001 0.001 0.0015; visual mesh filename=package://ur10/robotis_rh_p12_rn/visual/l2.stl scale=0.001 0.001 0.0015
- link rh_p12_rn_r1: geometry collision mesh filename=package://ur10/robotis_rh_p12_rn/collision/r1.stl scale=0.001 0.001 0.001; visual mesh filename=package://ur10/robotis_rh_p12_rn/visual/r1.stl scale=0.001 0.001 0.001
- link rh_p12_rn_r2: geometry collision mesh filename=package://ur10/robotis_rh_p12_rn/collision/r2.stl scale=0.001 0.001 0.0015; visual mesh filename=package://ur10/robotis_rh_p12_rn/visual/r2.stl scale=0.001 0.001 0.0015
- link shoulder_link: geometry collision mesh filename=package://ur10/ur10/collision/shoulder.stl; visual mesh filename=package://ur10/ur10/visual/shoulder.dae
- link upper_arm_link: geometry collision mesh filename=package://ur10/ur10/collision/upperarm.stl; visual mesh filename=package://ur10/ur10/visual/upperarm.dae
- link wrist_1_link: geometry collision mesh filename=package://ur10/ur10/collision/wrist1.stl; visual mesh filename=package://ur10/ur10/visual/wrist1.dae
- link wrist_2_link: geometry collision mesh filename=package://ur10/ur10/collision/wrist2.stl; visual mesh filename=package://ur10/ur10/visual/wrist2.dae
- link wrist_3_link: geometry collision mesh filename=package://ur10/ur10/collision/wrist3.stl; visual mesh filename=package://ur10/ur10/visual/wrist3.dae
