Commit message: update ur10 model

File: data/robots/ur10_klampt.urdf (robot description, URDF)
Before this commit: robot ur10_robotis_d435, 19 links, 18 joints
Links:
- added link world
Joints:
- added joint fied_world: type fixed, parent world, child base
- joint shoulder_pan_joint: limit lower=-1000 upper=1000 effort=330.0 velocity=2.16 -> lower=-6.283185307179586 upper=6.283185307179586 effort=330.0 velocity=2.16
- joint wrist_3_joint: limit lower=-1000 upper=1000 effort=54.0 velocity=3.2 -> lower=-6.283185307179586 upper=6.283185307179586 effort=54.0 velocity=3.2

File: data/robots/ur10_rod.urdf (robot description, URDF)
Before this commit: robot ur10_robotis_d435, 19 links, 18 joints
Links:
- removed link world
- added link base, mass 1e-3
- link base_link: geometry collision mesh filename=package://ur10/collision/base.stl; visual mesh filename=package://ur10/visual/base.obj
- link d435_link: geometry collision box size=0.02505 0.09 0.025; visual mesh filename=package://realsense2/visual/d435.obj
- link ee_link: mass 1e-3 -> 1e-2; geometry collision cylinder length=0.17 radius=0.01; visual cylinder length=0.17 radius=0.01
- link forearm_link: geometry collision mesh filename=package://ur10/collision/forearm.stl; visual mesh filename=package://ur10/visual/forearm.obj
- link rh_p12_rn_base: geometry collision mesh filename=package://robotis_rh_p12_rn/collision/base.stl scale=0.001 0.001 0.001; visual mesh filename=package://robotis_rh_p12_rn/visual/base.stl scale=0.001 0.001 0.001
- link rh_p12_rn_l1: geometry collision mesh filename=package://robotis_rh_p12_rn/collision/l1.stl scale=0.001 0.001 0.001; visual mesh filename=package://robotis_rh_p12_rn/visual/l1.stl scale=0.001 0.001 0.001
- link rh_p12_rn_l2: geometry collision mesh filename=package://robotis_rh_p12_rn/collision/l2.stl scale=0.001 0.001 0.001; visual mesh filename=package://robotis_rh_p12_rn/visual/l2.stl scale=0.001 0.001 0.001
- link rh_p12_rn_r1: geometry collision mesh filename=package://robotis_rh_p12_rn/collision/r1.stl scale=0.001 0.001 0.001; visual mesh filename=package://robotis_rh_p12_rn/visual/r1.stl scale=0.001 0.001 0.001
- link rh_p12_rn_r2: geometry collision mesh filename=package://robotis_rh_p12_rn/collision/r2.stl scale=0.001 0.001 0.001; visual mesh filename=package://robotis_rh_p12_rn/visual/r2.stl scale=0.001 0.001 0.001
- link shoulder_link: geometry collision mesh filename=package://ur10/collision/shoulder.stl; visual mesh filename=package://ur10/visual/shoulder.obj
- link upper_arm_link: geometry collision mesh filename=package://ur10/collision/upperarm.stl; visual mesh filename=package://ur10/visual/upperarm.obj
- link wrist_1_link: geometry collision mesh filename=package://ur10/collision/wrist1.stl; visual mesh filename=package://ur10/visual/wrist1.obj
- link wrist_2_link: geometry collision mesh filename=package://ur10/collision/wrist2.stl; visual mesh filename=package://ur10/visual/wrist2.obj
- link wrist_3_link: geometry collision mesh filename=package://ur10/collision/wrist3.stl; visual mesh filename=package://ur10/visual/wrist3.obj
Joints:
- removed joint fied_world
- added joint base_link-base_fixed_joint: type fixed, parent base, child base_link, origin xyz=0 0 0 rpy=0 0 -3.141592653589793
- joint d435_color_joint: origin xyz=0 0.015 0 rpy=0 0 0 -> xyz=-0.015 0 0 rpy=0 0 0
- joint d435_depth_joint: origin xyz=0 0 0 rpy=0 0 0 -> xyz=0 0 0 rpy=1.5707963267948966 0 1.5707963267948966
- joint d435_joint: origin xyz=-0.03 0 0.03 rpy=0 -1.57 0 -> xyz=-0.03 0 0.03 rpy=0 -1.5707963267948966 0
- joint ee_fixed_joint: origin xyz=0.0 0.0 0.135 rpy=0.0 0.0 0.0 -> xyz=0.0 0.0 0.260 rpy=0.0 0.0 0.0
- joint rh_l1: axis 0 1 0 -> -1 0 0; limit lower=0.0 upper=0.053 effort=1000 velocity=6.5 -> lower=0.95 upper=0.95 effort=1000 velocity=6.5; origin xyz=0.0 -0.008 0.048 rpy=0 0 0 -> xyz=0.0 -0.008 0.058 rpy=0 0 0; type prismatic -> revolute
- joint rh_l2: axis (none) -> 1 0 0; limit (none) -> lower=0.95 upper=0.95 effort=1000 velocity=6.5; mimic (none) -> joint=rh_p12_rn multiplier=1 offset=0; type fixed -> revolute
- joint rh_p12_rn: axis 0 -1 0 -> 1 0 0; limit lower=0.0 upper=0.053 effort=1000 velocity=6.5 -> lower=0.95 upper=0.95 effort=1000 velocity=6.5; origin xyz=0.0 0.008 0.048 rpy=0 0 0 -> xyz=0.0 0.008 0.058 rpy=0 0 0; type prismatic -> revolute
- joint rh_r2: axis (none) -> -1 0 0; limit (none) -> lower=0.95 upper=0.95 effort=1000 velocity=6.5; mimic (none) -> joint=rh_p12_rn multiplier=1 offset=0; type fixed -> revolute
- joint shoulder_pan_joint: limit lower=-6.283185307179586 upper=6.283185307179586 effort=330.0 velocity=2.16 -> lower=-1000 upper=1000 effort=330.0 velocity=2.16
- joint tool0_rh_p12_rn_base: origin xyz=0 0 0 rpy=0 0 0 -> xyz=0 0 0 rpy=0 0 -1.570796
- joint wrist_3_joint: limit lower=-6.283185307179586 upper=6.283185307179586 effort=54.0 velocity=3.2 -> lower=-1000 upper=1000 effort=54.0 velocity=3.2

File: data/robots/ur10_rod_klampt.urdf (robot description, URDF)
Before this commit: robot ur10_robotis_d435, 19 links, 18 joints
Links:
- added link world
- link ee_link: mass 1e-3 -> 1e-2; geometry collision cylinder length=0.17 radius=0.01; visual cylinder length=0.17 radius=0.01
Joints:
- added joint fied_world: type fixed, parent world, child base
- joint ee_fixed_joint: origin xyz=0.0 0.0 0.145 rpy=0.0 0.0 0.0 -> xyz=0.0 0.0 0.260 rpy=0.0 0.0 0.0
- joint rh_l1: limit lower=0.0 upper=1.12 effort=1000 velocity=6.5 -> lower=0.95 upper=0.95 effort=1000 velocity=6.5
- joint rh_l2: limit lower=0.0 upper=1.12 effort=1000 velocity=6.5 -> lower=0.95 upper=0.95 effort=1000 velocity=6.5
- joint rh_p12_rn: limit lower=0.0 upper=1.12 effort=1000 velocity=6.5 -> lower=0.95 upper=0.95 effort=1000 velocity=6.5
- joint rh_r2: limit lower=0.0 upper=1.12 effort=1000 velocity=6.5 -> lower=0.95 upper=0.95 effort=1000 velocity=6.5
- joint shoulder_pan_joint: limit lower=-1000 upper=1000 effort=330.0 velocity=2.16 -> lower=-6.283185307179586 upper=6.283185307179586 effort=330.0 velocity=2.16
- joint wrist_3_joint: limit lower=-1000 upper=1000 effort=54.0 velocity=3.2 -> lower=-6.283185307179586 upper=6.283185307179586 effort=54.0 velocity=3.2
